File: cyberdeck/k1/k1.kicad_pcb (KiCad board)
At the start: 2 copper layers, 98.8 x 94.7 mm, 73 parts, among them J1 Conn_01x20_MountingPin, J2 Conn_01x20_MountingPin, SW0 #0 ), SW1 #1 !, SW2 #2 @, SW3 #3 #, SW4 #4 $, SW5 #5 %, SW6 #6 ^, SW7 #7 &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

Commit message: posiblemente funcional
Parts:
- J1, J2: moved to B.Cu
- SWi1: value I | -> I }
- SWq1: value Q -> Q \
- SWu1: value U \ -> U {
- SWw1: value W -> W |
- moved J1 48.4 mm to (128.4, 65.0)
- moved J2 48.4 mm to (128.4, 47.2)
- moved RR3 3.27 mm to (176.7, 53.3)
- moved REF** 1.40 mm to (101.6, 47.2)
- moved REF** 1.40 mm to (192.5, 47.2)
Connections:
- J1 pad 1: unconnected-(J1-Pad1) -> c1
- J1 pad 10: c9 -> ledS
- J1 pad 11: c8 -> c7
- J1 pad 12: c7 -> ledC
- J1 pad 14: c6 -> c8
- J1 pad 15: c5 -> ledA
- J1 pad 16: c4 -> c9
- J1 pad 17: c3 -> cA
- J1 pad 19: c2 -> cB
- J1 pad 2: unconnected-(J1-Pad2) -> c2
- J1 pad 20: c1 -> cC
- J1 pad 4: unconnected-(J1-Pad4) -> c3
- J1 pad 5: unconnected-(J1-Pad5) -> c4
- J1 pad 6: cC -> c5
- J1 pad 7: cB -> ledF
- J1 pad 9: cA -> c6
- J2 pad 10: ledC -> Net-(RR4-Pad1)
- J2 pad 12: ledS -> Net-(RR5-Pad1)
- J2 pad 14: ledF -> unconnected-(J2-Pad14)
- J2 pad 15: Net-(J2-Pad15) -> unconnected-(J2-Pad15)
- J2 pad 16: Net-(J2-Pad16) -> unconnected-(J2-Pad16)
- J2 pad 19: Net-(RR1-Pad1) -> unconnected-(J2-Pad19)
- J2 pad 20: Net-(RR2-Pad1) -> Net-(RR3-Pad1)
- J2 pad 5: 3v3 -> unconnected-(J2-Pad5)
- J2 pad 7: Net-(RR3-Pad1) -> Net-(J2-Pad7)
- J2 pad 9: ledA -> Net-(J2-Pad9)
- RR1 pad 1: Net-(RR1-Pad1) -> Net-(J2-Pad9)
- RR2 pad 1: Net-(RR2-Pad1) -> Net-(J2-Pad7)
- RR4 pad 1: Net-(J2-Pad16) -> Net-(RR4-Pad1)
- RR5 pad 1: Net-(J2-Pad15) -> Net-(RR5-Pad1)
Routing:
- net r1: track 148.5 -> 227.9 mm
- net r2: track 162.7 -> 240.7 mm
- net r4: track 181.7 -> 259.7 mm
- net r3: track 151.2 -> 220.1 mm
- net r5: track 181.3 -> 226.8 mm
- net GND: track 35.6 -> 0.00 mm
- net c6: track 66.6 -> 101.7 mm
- net c2: track 74.6 -> 105.3 mm
- net c3: track 75.7 -> 104.3 mm
- net c7: track 55.0 -> 81.4 mm
- net Net-(J2-Pad7): track 0.00 -> 26.3 mm
- net c5: track 57.2 -> 83.3 mm
- net c1: track 74.9 -> 100.9 mm
- net Net-(J2-Pad9): track 0.00 -> 24.6 mm
- net Net-(RR5-Pad1): track 0.00 -> 23.7 mm
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Other:
- board size 98.8 x 94.7 mm -> 98.8 x 96.1 mm
- board text added: "GP00 P.1 C1"
- board text added: "GP01 P.2 C2"
- board text added: "GP02 P.4 C3"
- board text added: "GP03 P.5 C4"
- board text added: "GP04 P.6 C5"
- board text added: "GP05 P.7 LedFN"
- board text added: "GP06 P.9 C6"
- board text added: "GP07 P.10 LedShift"
- board text added: "GP09 P.12 LedCtrl"
- board text added: "GP10 P.14 C8"
- board text added: "GP12 P.15 LedAlt"
- board text added: "GP12 P.16 C9"
- board text added: "GP13 P.17 CA"
- board text added: "GP14 P.19 CB"
- board text added: "GP15 P.20 CC"
- board text added: "GP16 P.21 R3"
- board text added: "GP22 P.29 R5"
- board text added: "GP26 P.31 R4"
- board text added: "GP27 P.32 R1"
- board text added: "GP28 P.34 R2"
- board text added: "GP8 P.11 C7"
- board text added: "H: PRN SCR J: SCROLL LOCK"
- board text added: "S: INS D:HOME F:PGUP X: DEL C:END V:PGDOWN"
- board text added: "TAB"
- board text removed: "3v3"
- board text removed: "GP10 P.14 C6"
- board text removed: "GP11 P.15 C5"
- board text removed: "GP12 P.16 C4"
- board text removed: "GP13 P.17 C3"
- board text removed: "GP14 P.19 C2"
- board text removed: "GP15 P.20 C1"
- board text removed: "GP16 P.21 R2"
- board text removed: "GP17 P.22 R1"
- board text removed: "GP19 P.25 R4"
- board text removed: "GP20 P.26 R5"
- board text removed: "GP21 P.27 LedFN"
- board text removed: "GP22 P.29 LedShift"
- board text removed: "GP26 P.31 LedCtrl"
- board text removed: "GP27 P.32 LedAlt"
- board text removed: "GP28 P.34 R3"
- board text removed: "GP4 P.6 CC"
- board text removed: "GP5 P.7 CB"
- board text removed: "GP6 P.9 CA"
- board text removed: "GP7 P.10 C9"
- board text removed: "GP8 P.11 C8"
- board text removed: "GP9 P.12 C7"
- board text removed: "S: INS D:HOME F:PGUP X: DEL C:END V:PGDOWN H: PRINT SCREEN J: SCROLL LOCK"
- board text removed: "TAB⇆"
